Commit message: pan tilt on progress

File: urdf/pan_tilt.urdf (robot description, URDF)
Before this commit: robot pan_tilt, 3 links, 2 joints
Joints:
- joint pan_joint: limit lower=-3.14 upper=3.14 effort=300 velocity=0.1 -> lower=32 upper=120 effort=300 velocity=0.1
- joint tilt_joint: limit lower=-4.64 upper=-1.5 effort=300 velocity=0.1 -> lower=70 upper=185 effort=300 velocity=0.1

File: urdf/pan_tilt.xacro (robot description, xacro)
@@ -42,5 +42,5 @@
     <origin xyz="0 0 0.1"/>
     <axis xyz="0 0 1" />
-    <limit effort="300" velocity="0.1" lower="-3.14" upper="3.14"/>
+    <limit effort="300" velocity="0.1" lower="32" upper="120"/>
     <dynamics damping="50" friction="1"/>
   </joint>
@@ -68,5 +68,5 @@
     <origin xyz="0 0 0.2"/>
     <axis xyz="0 1 0" />
-    <limit effort="300" velocity="0.1" lower="-4.64" upper="-1.5"/>
+    <limit effort="300" velocity="0.1" lower="70" upper="185"/>
     <dynamics damping="50" friction="1"/>
   </joint>
